File: hardware/reflow-toaster-mainboard/reflow-toaster-mainboard.kicad_pcb (KiCad board)
At the start: 2 copper layers, 49.8 x 54.9 mm, 46 parts, among them J1 ili9481_tft_lcd, J2 Ext., J3 JTAG, J4 Speaker, J5 Door servo, J6 Thermocouple, J7 Serial, Q1 Si1308EDL, Q2 Si1308EDL, U1 STM32F103VDTx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

Commit message: Update PCB to KiCad v7
Other:
- net class Default removed
- net class Extra clearance removed
